File: Schematic/ManoMeter.sch (EAGLE design)
At the start: 14 parts, among them IC1 MPS20N0040D-S, U1 ADAFRUIT_ADS1115, X1 22-23-2021

Commit message: BlusDiodeToegevoegd
Parts:
- added D1: 1N4148DO35-10, diode:1N4148DO35-10
Connections:
- net GND: now also D1.A
- net N$11: now also D1.C
Changed lines of the file:
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@@
 <part name="GND5" library="supply1" deviceset="GND" device=""/>
 <part name="5" library="testpad" deviceset="PTR1" device="B1,27"/>
+<part name="D1" library="diode" deviceset="1N4148" device="DO35-10"/>
 </parts>
 <sheets>
@@
 <instance part="S1" gate="BEF1" x="104.14" y="134.62" rot="R90"/>
 <instance part="R1" gate="1" x="101.6" y="114.3" rot="R180"/>
-<instance part="Q1" gate="G$1" x="99.06" y="53.34"/>
+<instance part="Q1" gate="G$1" x="99.06" y="53.34" smashed="yes">
+<attribute name="NAME" x="96.52" y="58.42" size="1.778" layer="95"/>
+</instance>
 <instance part="U1" gate="G$1" x="106.68" y="180.34"/>
 <instance part="P+1" gate="VCC" x="88.9" y="208.28"/>
@@
 <instance part="GND5" gate="1" x="101.6" y="33.02"/>
 <instance part="5" gate="G$1" x="66.04" y="50.8" rot="R270"/>
+<instance part="D1" gate="G$1" x="109.22" y="53.34" smashed="yes" rot="R90">
+<attribute name="NAME" x="111.76" y="58.9026" size="1.778" layer="95"/>
+<attribute name="VALUE" x="111.76" y="56.1086" size="1.778" layer="96"/>
+</instance>
 </instances>
 <busses>
@@
 <pinref part="GND5" gate="1" pin="GND"/>
 <wire x1="91.44" y1="35.56" x2="101.6" y2="35.56" width="0.1524" layer="91"/>
-<wire x1="101.6" y1="35.56" x2="101.6" y2="48.26" width="0.1524" layer="91"/>
+<wire x1="101.6" y1="35.56" x2="101.6" y2="45.72" width="0.1524" layer="91"/>
 <junction x="101.6" y="35.56"/>
+<pinref part="D1" gate="G$1" pin="A"/>
+<wire x1="101.6" y1="45.72" x2="101.6" y2="48.26" width="0.1524" layer="91"/>
+<wire x1="109.22" y1="50.8" x2="109.22" y2="45.72" width="0.1524" layer="91"/>
+<wire x1="109.22" y1="45.72" x2="101.6" y2="45.72" width="0.1524" layer="91"/>
+<junction x="101.6" y="45.72"/>
 </segment>
 </net>
@@
 <pinref part="X1" gate="-2" pin="S"/>
 <wire x1="104.14" y1="66.04" x2="101.6" y2="66.04" width="0.1524" layer="91"/>
-<wire x1="101.6" y1="66.04" x2="101.6" y2="58.42" width="0.1524" layer="91"/>
+<wire x1="101.6" y1="66.04" x2="101.6" y2="60.96" width="0.1524" layer="91"/>
+<pinref part="D1" gate="G$1" pin="C"/>
+<wire x1="109.22" y1="55.88" x2="109.22" y2="60.96" width="0.1524" layer="91"/>
+<wire x1="109.22" y1="60.96" x2="101.6" y2="60.96" width="0.1524" layer="91"/>
+<wire x1="101.6" y1="60.96" x2="101.6" y2="58.42" width="0.1524" layer="91"/>
+<junction x="101.6" y="60.96"/>
 </segment>
 </net>

Commit message: PcbAdded
Parts:
- removed 12, 13, 5, 8, A0, SCL, SDA: PTR1B1,27, testpad:PTR1B1,27
- removed U1: ADAFRUIT_ADS1115, AD convertor:ADAFRUIT_ADS1115
- added C1, C16, C2: 10u, rcl:C-EUC1210
- added C14, C22, C24, C3: 100n, rcl:C-EUC0805
- added C15, C21, C25, C26: 100N, rcl:C-EUC0805
- added C17, C18: 22p, rcl:C-EUC0805
- added C19: 10uF, rcl:CPOL-EUR/2012-12R
- added FB1, FB2: MMZ2012Y152B, microbuilder:FERRITE0805
- added IC2: ATMEGA328P-32PIN-AU, avr:ATMEGA328P-32PIN-AU
- added IC3: CH340C, CH340C:CH340C
- added IC4: ADS1115IDGST, ADS1115IDGST:ADS1115IDGST
- added ISP: (no value), HR911105:HEADER-2X3P-SMD
- added K2: USB_MINI-B_SMT, SparkFun-Connectors:USB_MINI-B_SMT
- added L1: 10uH, microbuilder:INDUCTOR0805
- added R4, R5, R6: 4K7, rcl:R-EU_M0805
- added R47: 10K, rcl:R-EU_M0805
- added SJ5: (no value), microbuilder:SOLDERJUMPERREFLOW
- added X2: 16Mhz, adafruit:XTALNX5032
Connections:
- removed net N$5: IC1.OUT+, U1.A3
- new net +5V: C1.1, C14.2, C16.1, C19.+, C2.1, C22.2, C24.2, C3.2, FB1.P$1, FB1.P$2, IC1.IN+, IC2.VCC, IC2.VCC1, IC3.VCC, IC4.VDD, ISP.2, L1.2, R1.A, R4.2, R47.2, R5.2, R6.2, SJ5.2
- new net AGND: C1.2, C3.1, FB2.P$2, IC1.IN-, IC4.GND
- new net MISO: ISP.1
- new net MOSI: ISP.4
- new net N$12: IC2.(PCI20/XCK/T0)PD4, S1.O
- new net N$21: IC3.UD-, K2.D-
- new net N$22: C15.1, IC3.V3
- new net N$32: C26.1, IC2.AREF
- new net N$33: C25.1, IC3.!DTR
- new net N$34: IC3.UD+, K2.D+
- new net N$36: IC2.(PCI17/TXD)PD1, IC3.RXD
- new net N$37: K2.VBUS, SJ5.1
- new net N$40: C21.1, IC2.AVCC, L1.1
- new net N$46: IC2.(PCI16/RXD)PD0, IC3.TXD
- new net N$49: C18.1, IC2.PB6(XTAL1/TOSC1/PCI6), X2.P$2
- new net N$51: C17.1, IC2.PB7(XTAL2/TOSC2/PCI7), X2.P$1
- new net RESET: C25.2, IC2.PC6(/RESET/PCI14), ISP.5, R47.1
- new net SCLK: ISP.3
- net GND: now also C14.1, C15.2, C16.2, C17.2, C18.2, C19.-, C2.2, C21.2, C22.1, C24.1, C26.2, FB2.P$1, IC2.AGND, IC2.GND, IC2.GND1, IC3.GND, IC4.ADDR, ISP.6, K2.GND, K2.SHIELD; no longer IC1.IN-, U1.GND
- net N$1: now also IC2.(PCI18/INT0)PD2; no longer 12.TP
- net N$2: now also IC1.OUT+, IC4.AIN3; no longer 13.TP, S1.O
- net N$3: now also IC4.AIN2; no longer U1.A2
- net N$4: now also IC2.(PCI13/ADC5/SCL)PC5, IC4.SCL, R6.1; no longer SCL.TP, U1.SCL
- net N$6: now also IC2.(PCI12/ADC4/SDA)PC4, IC4.SDA, R5.1; no longer SDA.TP, U1.SDA
- net N$7: now also IC2.(PCI11/ADC3)PC3, IC4.ALERT/RDY, R4.1; no longer 8.TP, U1.ALRT
- net N$8: now also IC2.(PCI8/ADC0)PC0; no longer A0.TP
- net N$9: now also IC2.(PCI19/INT1/OC2B)PD3; no longer 5.TP
- net VCC: no longer IC1.IN+, R1.A, U1.VDD
Other:
- moved on the sheet: D1, IC1, Q1, R1, R2, R3, S1, X1-1, X1-2

Commit message: ChangedSensorType
Parts:
- removed IC1: MPS20N0040D-S, SparkFun-Connectors:MPS20N0040D-S
- added C4: 47p, rcl:C-EUC0805
- added IC5: MPXH6115AC6U, MPXH6115AC6U:MPXH6115AC6U
- added R7: 51K, rcl:R-EU_M0805
- C1: value 10u -> 100n; device rcl:C-EUC1210 -> rcl:C-EUC0805; FABRIKANTNO GRM32ER61A106KA01L -> (none)
Connections:
- removed net N$2: IC1.OUT+, IC4.AIN3
- removed net N$3: IC1.OUT-, IC1.OUT-2, IC4.AIN2
- new net N$5: C4.1, IC4.AIN3, IC5.VOUT, R7.2
- net +5V: now also C1.2, IC5.VS; no longer C1.1, IC1.IN+
- net AGND: now also C1.1, C4.2, IC5.GND, R7.1; no longer C1.2, IC1.IN-
Other:
- moved on the sheet: C1
Changed lines of the file:
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@@
 <part name="R1" library="pot" deviceset="TRIM_EU-" device="B25P" value="10K"/>
 <part name="Q1" library="transistor-power" deviceset="N-MOSFET_SYMBOL" device=""/>
-<part name="IC1" library="SparkFun-Connectors" deviceset="MPS20N0040D-S" device=""/>
 <part name="GND3" library="supply1" deviceset="GND" device=""/>
 <part name="X1" library="con-molex" deviceset="22-23-2021" device="" value=""/>
@@
 <part name="R5" library="rcl" deviceset="R-EU_" device="M0805" value="4K7"/>
 <part name="R6" library="rcl" deviceset="R-EU_" device="M0805" value="4K7"/>
-<part name="C1" library="rcl" deviceset="C-EU" device="C1210" value="10u">
-<attribute name="FABRIKANTNO" value="GRM32ER61A106KA01L"/>
-<attribute name="FARNELL" value=""/>
-</part>
 <part name="P+1" library="supply1" deviceset="+5V" device="" value="+5V AVDD"/>
 <part name="P+2" library="supply1" deviceset="+5V" device="" value="+5V AVDD"/>
@@
 <part name="SUPPLY6" library="supply2" deviceset="+5V" device=""/>
 <part name="P+3" library="supply1" deviceset="+5V" device="" value="+5V AVDD"/>
+<part name="IC5" library="MPXH6115AC6U" deviceset="MPXH6115AC6U" device=""/>
+<part name="C1" library="rcl" deviceset="C-EU" device="C0805" value="100n"/>
+<part name="C4" library="rcl" deviceset="C-EU" device="C0805" value="47p">
+<attribute name="FARNELL" value="1759489"/>
+</part>
+<part name="R7" library="rcl" deviceset="R-EU_" device="M0805" value="51K"/>
 </parts>
 <sheets>
@@
 <attribute name="NAME" x="269.24" y="134.62" size="1.778" layer="95"/>
 </instance>
-<instance part="IC1" gate="G$1" x="345.44" y="205.74"/>
 <instance part="GND3" gate="1" x="238.76" y="165.1"/>
 <instance part="X1" gate="-1" x="279.4" y="144.78"/>
@@
 <instance part="R5" gate="G$1" x="233.68" y="223.52" rot="R90"/>
 <instance part="R6" gate="G$1" x="238.76" y="223.52" rot="R90"/>
-<instance part="C1" gate="G$1" x="365.76" y="91.44">
-<attribute name="FABRIKANTNO" x="365.76" y="91.44" size="1.778" layer="96" display="off"/>
-<attribute name="FARNELL" x="365.76" y="91.44" size="1.778" layer="96" display="off"/>
-</instance>
 <instance part="P+1" gate="1" x="320.04" y="243.84"/>
 <instance part="P+2" gate="1" x="365.76" y="104.14"/>
@@
 <instance part="FB1" gate="G$1" x="332.74" y="96.52"/>
 <instance part="FB2" gate="G$1" x="332.74" y="83.82"/>
-<instance part="SUPPLY3" gate="G$1" x="342.9" y="182.88"/>
+<instance part="SUPPLY3" gate="G$1" x="325.12" y="160.02"/>
 <instance part="SUPPLY4" gate="G$1" x="342.9" y="78.74"/>
 <instance part="SUPPLY5" gate="G$1" x="365.76" y="78.74"/>
@@
 <instance part="SUPPLY6" gate="+5V" x="322.58" y="104.14"/>
 <instance part="P+3" gate="1" x="342.9" y="104.14"/>
+<instance part="IC5" gate="G$1" x="360.68" y="205.74" rot="R180"/>
+<instance part="C1" gate="G$1" x="365.76" y="88.9" smashed="yes" rot="R180">
+<attribute name="NAME" x="367.284" y="91.821" size="1.778" layer="95"/>
+<attribute name="VALUE" x="367.284" y="86.741" size="1.778" layer="96"/>
+</instance>
+<instance part="C4" gate="G$1" x="299.72" y="170.18">
+<attribute name="FARNELL" x="299.72" y="170.18" size="1.778" layer="96" display="off"/>
+</instance>
+<instance part="R7" gate="G$1" x="292.1" y="170.18" rot="R90"/>
 </instances>
 <busses>
@@
 <wire x1="276.86" y1="144.78" x2="274.32" y2="144.78" width="0.1524" layer="91"/>
 <wire x1="274.32" y1="144.78" x2="274.32" y2="154.94" width="0.1524" layer="91"/>
-</segment>
-</net>
-<net name="N$3" class="0">
-<segment>
-<pinref part="IC1" gate="G$1" pin="OUT-"/>
-<wire x1="330.2" y1="210.82" x2="327.66" y2="210.82" width="0.1524" layer="91"/>
-<wire x1="327.66" y1="210.82" x2="320.04" y2="210.82" width="0.1524" layer="91"/>
-<pinref part="IC1" gate="G$1" pin="OUT-2"/>
-<wire x1="360.68" y1="210.82" x2="368.3" y2="210.82" width="0.1524" layer="91"/>
-<wire x1="368.3" y1="210.82" x2="368.3" y2="218.44" width="0.1524" layer="91"/>
-<wire x1="368.3" y1="218.44" x2="327.66" y2="218.44" width="0.1524" layer="91"/>
-<wire x1="327.66" y1="218.44" x2="327.66" y2="210.82" width="0.1524" layer="91"/>
-<junction x="327.66" y="210.82"/>
-<wire x1="320.04" y1="210.82" x2="320.04" y2="177.8" width="0.1524" layer="91"/>
-<wire x1="320.04" y1="177.8" x2="269.24" y2="177.8" width="0.1524" layer="91"/>
-<wire x1="269.24" y1="177.8" x2="269.24" y2="208.28" width="0.1524" layer="91"/>
-<pinref part="IC4" gate="A" pin="AIN2"/>
-<wire x1="269.24" y1="208.28" x2="276.86" y2="208.28" width="0.1524" layer="91"/>
 </segment>
 </net>
@@
 <wire x1="317.5" y1="220.98" x2="317.5" y2="233.68" width="0.1524" layer="91"/>
 <wire x1="322.58" y1="233.68" x2="320.04" y2="233.68" width="0.1524" layer="91"/>
-<pinref part="IC1" gate="G$1" pin="IN+"/>
 <wire x1="320.04" y1="233.68" x2="317.5" y2="233.68" width="0.1524" layer="91"/>
-<wire x1="330.2" y1="205.74" x2="322.58" y2="205.74" width="0.1524" layer="91"/>
-<wire x1="322.58" y1="205.74" x2="322.58" y2="233.68" width="0.1524" layer="91"/>
 <pinref part="P+1" gate="1" pin="+5V"/>
 <wire x1="320.04" y1="233.68" x2="320.04" y2="241.3" width="0.1524" layer="91"/>
 <junction x="320.04" y="233.68"/>
-</segment>
-<segment>
-<pinref part="C1" gate="G$1" pin="1"/>
+<pinref part="IC5" gate="G$1" pin="VS"/>
+<wire x1="330.2" y1="210.82" x2="317.5" y2="210.82" width="0.1524" layer="91"/>
+<wire x1="317.5" y1="210.82" x2="317.5" y2="220.98" width="0.1524" layer="91"/>
+<junction x="317.5" y="220.98"/>
+</segment>
+<segment>
 <wire x1="365.76" y1="93.98" x2="365.76" y2="101.6" width="0.1524" layer="91"/>
 <pinref part="P+2" gate="1" pin="+5V"/>
+<pinref part="C1" gate="G$1" pin="2"/>
 </segment>
 <segment>
@@
 </segment>
 </net>
-<net name="N$2" class="0">
-<segment>
-<pinref part="IC1" gate="G$1" pin="OUT+"/>
-<wire x1="330.2" y1="200.66" x2="322.58" y2="200.66" width="0.1524" layer="91"/>
-<wire x1="322.58" y1="200.66" x2="322.58" y2="175.26" width="0.1524" layer="91"/>
-<wire x1="322.58" y1="175.26" x2="271.78" y2="175.26" width="0.1524" layer="91"/>
-<wire x1="271.78" y1="175.26" x2="271.78" y2="205.74" width="0.1524" layer="91"/>
-<pinref part="IC4" gate="A" pin="AIN3"/>
-<wire x1="271.78" y1="205.74" x2="276.86" y2="205.74" width="0.1524" layer="91"/>
-</segment>
-</net>
 <net name="AGND" class="0">
 <segment>
+<pinref part="SUPPLY3" gate="G$1" pin="AGND"/>
+<pinref part="IC5" gate="G$1" pin="GND"/>
+<wire x1="330.2" y1="208.28" x2="325.12" y2="208.28" width="0.1524" layer="91"/>
+<wire x1="325.12" y1="208.28" x2="325.12" y2="190.5" width="0.1524" layer="91"/>
 <pinref part="IC4" gate="A" pin="GND"/>
-<wire x1="312.42" y1="190.5" x2="314.96" y2="190.5" width="0.1524" layer="91"/>
-<wire x1="314.96" y1="190.5" x2="314.96" y2="185.42" width="0.1524" layer="91"/>
-<pinref part="IC1" gate="G$1" pin="IN-"/>
-<wire x1="360.68" y1="205.74" x2="368.3" y2="205.74" width="0.1524" layer="91"/>
-<wire x1="368.3" y1="205.74" x2="368.3" y2="185.42" width="0.1524" layer="91"/>
-<wire x1="314.96" y1="185.42" x2="342.9" y2="185.42" width="0.1524" layer="91"/>
-<pinref part="SUPPLY3" gate="G$1" pin="AGND"/>
-<wire x1="342.9" y1="185.42" x2="368.3" y2="185.42" width="0.1524" layer="91"/>
-<junction x="342.9" y="185.42"/>
-</segment>
-<segment>
-<pinref part="C1" gate="G$1" pin="2"/>
+<wire x1="325.12" y1="190.5" x2="325.12" y2="162.56" width="0.1524" layer="91"/>
+<wire x1="312.42" y1="190.5" x2="325.12" y2="190.5" width="0.1524" layer="91"/>
+<junction x="325.12" y="190.5"/>
+<pinref part="R7" gate="G$1" pin="1"/>
+<wire x1="292.1" y1="165.1" x2="292.1" y2="162.56" width="0.1524" layer="91"/>
+<wire x1="292.1" y1="162.56" x2="299.72" y2="162.56" width="0.1524" layer="91"/>
+<pinref part="C4" gate="G$1" pin="2"/>
+<wire x1="299.72" y1="162.56" x2="325.12" y2="162.56" width="0.1524" layer="91"/>
+<wire x1="299.72" y1="165.1" x2="299.72" y2="162.56" width="0.1524" layer="91"/>
+<junction x="299.72" y="162.56"/>
+<junction x="325.12" y="162.56"/>
+</segment>
+<segment>
 <wire x1="365.76" y1="86.36" x2="365.76" y2="81.28" width="0.1524" layer="91"/>
 <pinref part="SUPPLY5" gate="G$1" pin="AGND"/>
+<pinref part="C1" gate="G$1" pin="1"/>
 </segment>
 <segment>
@@
 </segment>
 </net>
+<net name="N$5" class="0">
+<segment>
+<pinref part="R7" gate="G$1" pin="2"/>
+<pinref part="IC4" gate="A" pin="AIN3"/>
+<wire x1="271.78" y1="205.74" x2="276.86" y2="205.74" width="0.1524" layer="91"/>
+<wire x1="271.78" y1="175.26" x2="271.78" y2="205.74" width="0.1524" layer="91"/>
+<wire x1="271.78" y1="175.26" x2="292.1" y2="175.26" width="0.1524" layer="91"/>
+<wire x1="320.04" y1="205.74" x2="320.04" y2="175.26" width="0.1524" layer="91"/>
+<pinref part="IC5" gate="G$1" pin="VOUT"/>
+<wire x1="320.04" y1="205.74" x2="330.2" y2="205.74" width="0.1524" layer="91"/>
+<wire x1="292.1" y1="175.26" x2="299.72" y2="175.26" width="0.1524" layer="91"/>
+<pinref part="C4" gate="G$1" pin="1"/>
+<wire x1="299.72" y1="175.26" x2="320.04" y2="175.26" width="0.1524" layer="91"/>
+<wire x1="299.72" y1="172.72" x2="299.72" y2="175.26" width="0.1524" layer="91"/>
+<junction x="292.1" y="175.26"/>
+<junction x="299.72" y="175.26"/>
+</segment>
+</net>

Commit message: AddedLibrary
Parts:
- removed D1: 1N4148DO35-10, diode:1N4148DO35-10
- removed K2: USB_MINI-B_SMT, SparkFun-Connectors:USB_MINI-B_SMT
- removed SJ5: (no value), microbuilder:SOLDERJUMPERREFLOW
- added D2: 1N4148SMD, Evert:1N4148SMD
- added JP1: USB-B, SparkFun-Connectors:USBPTH
- R2, R3: device rcl:R-EU_0204/5 -> rcl:R-EU_M0805
Connections:
- removed net N$37: K2.VBUS, SJ5.1
- net +5V: now also JP1.VBUS; no longer SJ5.2
- net GND: now also JP1.GND, JP1.GND1, JP1.GND2; no longer D1.A, K2.GND, K2.SHIELD
- net N$11: no longer D1.C
- net N$21: now also JP1.D-; no longer K2.D-
- net N$34: now also JP1.D+; no longer K2.D+
Changed lines of the file:
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@@
 <part name="X1" library="con-molex" deviceset="22-23-2021" device="" value=""/>
 <part name="SUPPLY1" library="supply2" deviceset="VCC" device="" value="+12V"/>
-<part name="R2" library="rcl" deviceset="R-EU_" device="0204/5" value="390"/>
-<part name="R3" library="rcl" deviceset="R-EU_" device="0204/5" value="1k"/>
+<part name="R2" library="rcl" deviceset="R-EU_" device="M0805" value="390"/>
+<part name="R3" library="rcl" deviceset="R-EU_" device="M0805" value="1k"/>
 <part name="GND5" library="supply1" deviceset="GND" device=""/>
-<part name="D1" library="diode" deviceset="1N4148" device="DO35-10"/>
 <part name="IC2" library="avr" deviceset="ATMEGA328P-32PIN" device="-AU">
 <attribute name="FARNELL" value="1972086"/>
@@
 <part name="C19" library="rcl" deviceset="CPOL-EU" device="R/2012-12R" value="10uF"/>
 <part name="GND12" library="supply1" deviceset="GND" device=""/>
-<part name="K2" library="SparkFun-Connectors" deviceset="USB_MINI-B" device="_SMT">
-<attribute name="FARNELL" value="1753806"/>
-</part>
 <part name="L1" library="microbuilder" deviceset="INDUCTOR" device="0805" value="10uH">
 <attribute name="FARNELL" value="2215650"/>
@@
 </part>
 <part name="SUPPLY13" library="supply2" deviceset="+5V" device=""/>
-<part name="SJ5" library="microbuilder" deviceset="SOLDERJUMPER" device="REFLOW"/>
 <part name="SUPPLY2" library="supply2" deviceset="+5V" device=""/>
 <part name="IC4" library="ADS1115IDGST" deviceset="ADS1115IDGST" device=""/>
@@
 </part>
 <part name="R7" library="rcl" deviceset="R-EU_" device="M0805" value="51K"/>
+<part name="D2" library="Evert" deviceset="1N4148" device="SMD"/>
+<part name="JP1" library="SparkFun-Connectors" deviceset="USB" device="PTH" value="USB-B"/>
 </parts>
 <sheets>
@@
 <instance part="R3" gate="G$1" x="264.16" y="119.38" rot="R90"/>
 <instance part="GND5" gate="1" x="274.32" y="109.22"/>
-<instance part="D1" gate="G$1" x="281.94" y="129.54" smashed="yes" rot="R90">
-<attribute name="NAME" x="284.48" y="135.1026" size="1.778" layer="95"/>
-<attribute name="VALUE" x="284.48" y="132.3086" size="1.778" layer="96"/>
-</instance>
 <instance part="IC2" gate="G$1" x="182.88" y="175.26">
 <attribute name="FARNELL" x="182.88" y="175.26" size="1.778" layer="96" display="off"/>
@@
 <instance part="C19" gate="G$1" x="157.48" y="96.52"/>
 <instance part="GND12" gate="1" x="162.56" y="81.28"/>
-<instance part="K2" gate="G$1" x="27.94" y="160.02">
-<attribute name="FARNELL" x="27.94" y="160.02" size="1.778" layer="96" display="off"/>
-</instance>
 <instance part="L1" gate="G$1" x="124.46" y="213.36" rot="R90">
 <attribute name="FARNELL" x="124.46" y="213.36" size="1.778" layer="96" rot="R90" display="off"/>
@@
 </instance>
 <instance part="SUPPLY13" gate="+5V" x="35.56" y="226.06"/>
-<instance part="SJ5" gate="1" x="35.56" y="180.34" rot="R90"/>
 <instance part="SUPPLY2" gate="+5V" x="274.32" y="243.84"/>
 <instance part="IC4" gate="A" x="294.64" y="205.74"/>
@@
 </instance>
 <instance part="R7" gate="G$1" x="292.1" y="170.18" rot="R90"/>
+<instance part="D2" gate="G$1" x="281.94" y="129.54" rot="R90"/>
+<instance part="JP1" gate="G$1" x="30.48" y="157.48" rot="MR0"/>
 </instances>
 <busses>
@@
 <wire x1="274.32" y1="111.76" x2="274.32" y2="121.92" width="0.1524" layer="91"/>
 <junction x="274.32" y="111.76"/>
-<pinref part="D1" gate="G$1" pin="A"/>
 <wire x1="274.32" y1="121.92" x2="274.32" y2="124.46" width="0.1524" layer="91"/>
 <wire x1="281.94" y1="127" x2="281.94" y2="121.92" width="0.1524" layer="91"/>
@@
 <wire x1="58.42" y1="142.24" x2="63.5" y2="142.24" width="0.1524" layer="91"/>
 <junction x="58.42" y="142.24"/>
-<pinref part="K2" gate="G$1" pin="GND"/>
-<wire x1="33.02" y1="157.48" x2="38.1" y2="157.48" width="0.1524" layer="91"/>
-<wire x1="38.1" y1="157.48" x2="38.1" y2="154.94" width="0.1524" layer="91"/>
-<pinref part="K2" gate="G$1" pin="SHIELD"/>
-<wire x1="33.02" y1="154.94" x2="38.1" y2="154.94" width="0.1524" layer="91"/>
-<junction x="38.1" y="154.94"/>
-<wire x1="38.1" y1="154.94" x2="38.1" y2="142.24" width="0.1524" layer="91"/>
-<wire x1="38.1" y1="142.24" x2="50.8" y2="142.24" width="0.1524" layer="91"/>
+<wire x1="35.56" y1="142.24" x2="50.8" y2="142.24" width="0.1524" layer="91"/>
 <junction x="50.8" y="142.24"/>
+<pinref part="JP1" gate="G$1" pin="GND"/>
+<wire x1="33.02" y1="157.48" x2="35.56" y2="157.48" width="0.1524" layer="91"/>
+<wire x1="35.56" y1="157.48" x2="35.56" y2="142.24" width="0.1524" layer="91"/>
+<pinref part="JP1" gate="G$1" pin="GND2"/>
+<wire x1="35.56" y1="142.24" x2="27.94" y2="142.24" width="0.1524" layer="91"/>
+<wire x1="27.94" y1="142.24" x2="25.4" y2="142.24" width="0.1524" layer="91"/>
+<wire x1="25.4" y1="142.24" x2="25.4" y2="152.4" width="0.1524" layer="91"/>
+<pinref part="JP1" gate="G$1" pin="GND1"/>
+<wire x1="27.94" y1="152.4" x2="27.94" y2="142.24" width="0.1524" layer="91"/>
+<junction x="27.94" y="142.24"/>
+<junction x="35.56" y="142.24"/>
 </segment>
 <segment>
@@
 <wire x1="276.86" y1="142.24" x2="274.32" y2="142.24" width="0.1524" layer="91"/>
 <wire x1="274.32" y1="142.24" x2="274.32" y2="137.16" width="0.1524" layer="91"/>
-<pinref part="D1" gate="G$1" pin="C"/>
 <wire x1="281.94" y1="132.08" x2="281.94" y2="137.16" width="0.1524" layer="91"/>
 <wire x1="281.94" y1="137.16" x2="274.32" y2="137.16" width="0.1524" layer="91"/>
@@
 <segment>
 <pinref part="SUPPLY13" gate="+5V" pin="+5V"/>
-<pinref part="SJ5" gate="1" pin="2"/>
-<wire x1="35.56" y1="223.52" x2="35.56" y2="185.42" width="0.1524" layer="91"/>
+<wire x1="35.56" y1="223.52" x2="35.56" y2="160.02" width="0.1524" layer="91"/>
+<pinref part="JP1" gate="G$1" pin="VBUS"/>
+<wire x1="33.02" y1="160.02" x2="35.56" y2="160.02" width="0.1524" layer="91"/>
 </segment>
 <segment>
@@
 <net name="N$21" class="0">
 <segment>
-<pinref part="K2" gate="G$1" pin="D-"/>
-<wire x1="33.02" y1="165.1" x2="40.64" y2="165.1" width="0.1524" layer="91"/>
-<wire x1="40.64" y1="165.1" x2="43.18" y2="162.56" width="0.1524" layer="91"/>
 <pinref part="IC3" gate="G$1" pin="UD-"/>
-<wire x1="43.18" y1="162.56" x2="63.5" y2="162.56" width="0.1524" layer="91"/>
+<wire x1="33.02" y1="162.56" x2="63.5" y2="162.56" width="0.1524" layer="91"/>
+<pinref part="JP1" gate="G$1" pin="D-"/>
 </segment>
 </net>
 <net name="N$34" class="0">
 <segment>
-<pinref part="K2" gate="G$1" pin="D+"/>
-<wire x1="33.02" y1="162.56" x2="40.64" y2="162.56" width="0.1524" layer="91"/>
-<wire x1="40.64" y1="162.56" x2="43.18" y2="165.1" width="0.1524" layer="91"/>
 <pinref part="IC3" gate="G$1" pin="UD+"/>
-<wire x1="43.18" y1="165.1" x2="63.5" y2="165.1" width="0.1524" layer="91"/>
+<wire x1="33.02" y1="165.1" x2="63.5" y2="165.1" width="0.1524" layer="91"/>
+<pinref part="JP1" gate="G$1" pin="D+"/>
 </segment>
 </net>
@@
 </segment>
 </net>
-<net name="N$37" class="0">
-<segment>
-<pinref part="SJ5" gate="1" pin="1"/>
-<wire x1="35.56" y1="175.26" x2="35.56" y2="167.64" width="0.1524" layer="91"/>
-<pinref part="K2" gate="G$1" pin="VBUS"/>
-<wire x1="35.56" y1="167.64" x2="33.02" y2="167.64" width="0.1524" layer="91"/>
-</segment>
-</net>
